File: minimal_adp1032/minimal_adp1032.kicad_pcb (KiCad board)
At the start: 4 copper layers, 34.3 x 38.1 mm, 58 parts, among them T1 ZA9644-AED, U1 ADP1032ACPZ-5-R7

Commit message: development backup
Parts:
- moved kibuzzard-6778FAD8 0.64 mm to (141.7, 118.7)
- moved kibuzzard-6778FC4F 0.64 mm to (165.6, 118.7)
- moved kibuzzard-6778F9B2 0.63 mm to (165.0, 87.0)
- moved kibuzzard-677D932A 0.63 mm to (142.1, 87.0)
Connections:
- net /ADP1032_VOUT1 renamed /VOUT1
Routing:
- net GNDD: vias 106 -> 57
- net GNDA: vias 66 -> 91
- net GND: vias 9 -> 31

Commit message: development backup
Parts:
- removed kibuzzard-6778F9B2: G***, kibuzzard-6778F9B2
- removed kibuzzard-6778FAD8: G***, kibuzzard-6778FAD8
- removed kibuzzard-6778FC4F: G***, kibuzzard-6778FC4F
- removed kibuzzard-677D932A: G***, kibuzzard-677D932A
- added kibuzzard-6780FB3F: G***, kibuzzard-6780FB3F, F.Cu at (146.1, 116.0)
- added kibuzzard-6780FE33: G***, kibuzzard-6780FE33, F.Cu at (146.1, 89.7)
- added kibuzzard-6780FE43: G***, kibuzzard-6780FE43, F.Cu at (161.3, 89.7)
- added kibuzzard-6781023F: G***, kibuzzard-6781023F, F.Cu at (161.3, 116.0)
- added kibuzzard-67810269: G***, kibuzzard-67810269, F.Cu at (156.8, 116.2)
- added kibuzzard-67810269: G***, kibuzzard-67810269, F.Cu at (150.5, 116.2)
- added kibuzzard-67810279: G***, kibuzzard-67810279, F.Cu at (141.6, 116.5)
- added kibuzzard-67810279: G***, kibuzzard-67810279, F.Cu at (165.7, 116.5)
- added kibuzzard-67810360: G***, kibuzzard-67810360, F.Cu at (165.7, 89.3)
- added kibuzzard-6781036E: G***, kibuzzard-6781036E, F.Cu at (141.6, 88.9)
- added kibuzzard-6781036E: G***, kibuzzard-6781036E, F.Cu at (156.8, 88.9)
- added kibuzzard-678103F7: G***, kibuzzard-678103F7, F.Cu at (150.5, 89.3)
- moved TP15 5.24 mm to (142.2, 120.6)
- moved TP18 5.24 mm to (142.2, 85.1)
- moved TP27 5.24 mm to (165.1, 120.6)
- moved TP30 5.24 mm to (165.1, 85.1)
- moved TP20 2.71 mm to (147.3, 119.0)
- moved TP21 2.71 mm to (147.3, 86.7)
- moved TP16 2.71 mm to (144.8, 119.0)
- moved TP17 2.71 mm to (144.8, 86.7)
- moved TP24 2.71 mm to (160.0, 119.0)
- moved TP25 2.71 mm to (160.0, 86.7)
- moved TP28 2.71 mm to (162.6, 119.0)
- moved TP29 2.71 mm to (162.6, 86.7)
- moved JP1 1.60 mm to (152.4, 117.2)
- moved JP2 1.60 mm to (154.9, 117.2)
- moved TP23 1.27 mm to (157.5, 120.6)
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Routing:
- net GNDD: vias 57 -> 49
- net GNDA: vias 91 -> 72
- net GND: vias 31 -> 23
- net /VINP: vias 5 -> 13
Other:
- board size 34.3 x 38.1 mm -> 34.3 x 35.6 mm
