File: minimal_adp1032/minimal_adp1032.kicad_sch (KiCad schematic)
At the start: 54 parts, among them T1 ZA9644-AED, U1 ADP1032ACPZ-5-R7

Commit message: development backup
Connections:
- net ADP1032_VOUT1 renamed VOUT1
Changed lines of the file:
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@@
-	)
-	(junction
-		(at 160.02 152.4)
-		(diameter 0)
-		(color 0 0 0 0)
 	)
 	(junction
@@
 	(wire
 		(pts
-			(xy 152.4 152.4) (xy 160.02 152.4)
-		)
-		(stroke
-			(width 0)
-			(type default)
-		)
-	)
-	(wire
-		(pts
 			(xy 312.42 222.25) (xy 312.42 224.79)
 		)
@@
 	(wire
 		(pts
-			(xy 309.88 86.36) (xy 330.2 86.36)
+			(xy 309.88 86.36) (xy 320.04 86.36)
 		)
 		(stroke
@@
 	(wire
 		(pts
-			(xy 309.88 127) (xy 330.2 127)
+			(xy 309.88 127) (xy 320.04 127)
 		)
 		(stroke
@@
 		)
 	)
-	(label "ADP1032_VOUT1"
-		(at 293.37 86.36 180)
-		(fields_autoplaced yes)
-		(effects
-			(font
-				(size 1.27 1.27)
-			)
-			(justify right bottom)
+	(label "VOUT1"
+		(at 283.21 86.36 0)
+		(fields_autoplaced yes)
+		(effects
+			(font
+				(size 1.27 1.27)
+			)
+			(justify left bottom)
 		)
 	)
@@
 	)
 	(label "VDD_24V"
-		(at 327.66 86.36 180)
+		(at 320.04 86.36 180)
 		(fields_autoplaced yes)
 		(effects
@@
 	)
 	(label "3V3_ISO"
-		(at 327.66 127 180)
+		(at 320.04 127 180)
 		(fields_autoplaced yes)
 		(effects
@@
 		)
 	)
-	(hierarchical_label "3V3_ISO"
-		(shape output)
-		(at 330.2 127 0)
-		(fields_autoplaced yes)
-		(effects
-			(font
-				(size 1.27 1.27)
-				(thickness 0.254)
-				(bold yes)
-			)
-			(justify left)
-		)
-	)
-	(hierarchical_label "VDD_24V"
-		(shape output)
-		(at 330.2 86.36 0)
-		(fields_autoplaced yes)
-		(effects
-			(font
-				(size 1.27 1.27)
-				(thickness 0.254)
-				(bold yes)
-			)
-			(justify left)
-		)
-	)
-	(hierarchical_label "MVDD"
-		(shape input)
-		(at 152.4 152.4 180)
-		(fields_autoplaced yes)
-		(effects
-			(font
-				(size 1.27 1.27)
-				(thickness 0.254)
-				(bold yes)
-			)
-			(justify right)
-		)
-	)

Commit message: change form factor to be more compact
Parts:
- removed TP16, TP17, TP20, TP21, TP24, TP25, TP28, TP29: TestPoint, test_point_footprints:TestPoint_THTPad_2.0x2.0mm_Drill1.0mm, symbol UNITED_TEST_POINTS:TestPoint
